File: 6502.kicad_pcb (KiCad board)
At the start: 2 copper layers, 95.2 x 95.3 mm, 38 parts, among them J3 Conn_01x40, J4 CPU Control, SW1 Reset, U1 W65C02SxP, U2 AT28C256, U3 HM62256BLP, Y1 1MHz

Commit message: Replace back-plane connector
Parts:
- removed J3: Conn_01x40, Connector_PinHeader_2.54mm:PinHeader_1x37_P2.54mm_Vertical
- removed REF** (x4): DIP-14_W7.62mm_Socket, Package_DIP:DIP-14_W7.62mm_Socket
- removed TP10, TP7, TP8, TP9: GND, TestPoint:TestPoint_Pad_D1.5mm
- removed TP3, TP4, TP5, TP6: +5V, TestPoint:TestPoint_Pad_D1.5mm
- added J1: ~, Connector_PinHeader_2.54mm:PinHeader_1x37_P2.54mm_Vertical, F.Cu at (61.6, 172.1)
Routing:
- net +5V: track 383.0 -> 293.1 mm, vias 9 -> 4

Commit message: Status LEDs
Parts:
- added D1: LED, LED_THT:LED_D3.0mm_Horizontal_O1.27mm_Z2.0mm, F.Cu at (65.4, 88.3)
- added D2: LED, LED_THT:LED_D3.0mm_Horizontal_O1.27mm_Z2.0mm, F.Cu at (71.8, 88.3)
- added R7: 10k, Resistor_SMD:R_1206_3216Metric, F.Cu at (62.9, 92.7)
- added R8: 10k, Resistor_SMD:R_1206_3216Metric, F.Cu at (69.2, 92.7)
Routing:
- net +5V: track 293.1 -> 309.6 mm
- net CPU_VPB: track 9.20 -> 25.3 mm
- net CPU_SYNC: track 32.5 -> 35.8 mm
- net Net-(D2-A): track 0.00 -> 2.98 mm
- net Net-(D1-A): track 0.00 -> 2.98 mm
Other:
- board text added: "TODO GH Url"
- board text added: "VP"
